Commit message: updated urdf and script for Spidey_V3

File: spidey_simulation/spidey_py/spidey_python/ik_solver/spidey_assets/urdf_and_meshes_v3/spidey_v3.urdf (robot description, URDF)
Before this commit: robot spidey, 17 links, 16 joints
Links:
- link base_link: mass 0.055807 -> 0.117924372960691
- link leg1_link1: mass 0.0072387 -> 0.00723872418872688
- link leg1_link2: mass 0.01229 -> 0.0122900929113511
- link leg1_link3: mass 0.016854 -> 0.0168535864832978
- link leg1_link3_tip: mass 9.9084E-07 -> 9.90841781413794E-07
- link leg2_link1: mass 0.0072387 -> 0.00723872418872687
- link leg2_link2: mass 0.01229 -> 0.0122900929113511
- link leg2_link3: mass 0.016854 -> 0.0168535864832979
- link leg2_link3_tip: mass 9.9084E-07 -> 9.90841781413787E-07
- link leg3_link1: mass 0.0072387 -> 0.00723872418872689
- link leg3_link2: mass 0.01229 -> 0.0122900929113511
- link leg3_link3: mass 0.016854 -> 0.0168535864832979
- link leg3_link3_tip: mass 9.9084E-07 -> 9.9084178141379E-07
- link leg4_link1: mass 0.0072387 -> 0.00723872418872688
- link leg4_link2: mass 0.01229 -> 0.0122900929113511
- link leg4_link3: mass 0.016854 -> 0.0168535864832979
- link leg4_link3_tip: mass 9.9084E-07 -> 9.90841781413788E-07
Joints:
- joint leg1_joint1: origin xyz=0.038964 -0.038964 0.0821 rpy=-1.5708 0 2.3562 -> xyz=0.046464 -0.046464 0.0821 rpy=-1.5708 0 2.3562
- joint leg2_joint1: origin xyz=0.038964 0.038964 0.0821 rpy=-1.5708 0 -2.3562 -> xyz=0.046464 0.046464 0.0821 rpy=-1.5708 0 -2.3562
- joint leg3_joint1: origin xyz=-0.038964 -0.038964 0.0821 rpy=-1.5708 0 0.7854 -> xyz=-0.046464 -0.046464 0.0821 rpy=-1.5708 0 0.7854
- joint leg3_joint2: origin xyz=-0.033 -0.0145 0 rpy=0 0 -3.1416 -> xyz=-0.033 -0.0145 0 rpy=0 0 3.1416
- joint leg4_joint1: origin xyz=-0.038964 0.038964 0.0821 rpy=-1.5708 0 -0.7854 -> xyz=-0.046464 0.046464 0.0821 rpy=-1.5708 0 -0.7854
- joint leg4_joint2: origin xyz=-0.033 -0.0145 0 rpy=0 0 -3.1416 -> xyz=-0.033 -0.0145 0 rpy=0 0 3.1416
